Commit message: fixed baseline on wback wheels

File: src/iwalk_description/urdf/iwalk.urdf.xacro (robot description, xacro)
@@ -5,17 +5,14 @@
   <!-- ==================================================== -->
   <!-- ΒΑΣΙΚΕΣ ΠΑΡΑΜΕΤΡΟΙ                                  -->
-  <!-- Οι παρακάτω αριθμοί είναι προσωρινοί.                -->
-  <!-- Θα αντικατασταθούν με μετρήσεις του πραγματικού      -->
-  <!-- i-Walk και του STL.                                  -->
   <!-- ==================================================== -->
   <xacro:property name="PI" value="3.141592653589793"/>
   <!-- Σταθερό ύψος του base_link από το έδαφος -->
-  <xacro:property name="base_link_height" value="0.10"/>
+  <xacro:property name="base_link_height" value="0.095"/>
   <!-- 0.001 αν το STL είναι σε mm, 1.0 αν είναι σε m -->
   <xacro:property name="mesh_scale" value="0.001"/>
   <!-- Μετατόπιση και περιστροφή του STL ως προς base_link -->
-  <xacro:property name="mesh_x" value="0.292367371"/>
+  <xacro:property name="mesh_x" value="0.682367371"/>
   <xacro:property name="mesh_y" value="-0.326500000"/>
-  <xacro:property name="mesh_z" value="-0.100114396"/>
+  <xacro:property name="mesh_z" value="-0.095114396"/>
   <xacro:property name="mesh_roll"  value="0.0"/>
   <xacro:property name="mesh_pitch" value="0.0"/>
@@ -24,7 +21,7 @@
   <xacro:property name="body_width"  value="0.653000000"/>
   <xacro:property name="body_height" value="1.046494491"/>
-  <xacro:property name="body_center_x" value="0.0"/>
+  <xacro:property name="body_center_x" value="0.39"/>
   <xacro:property name="body_center_y" value="0.0"/>
-  <xacro:property name="body_center_z" value="0.423247245"/>
+  <xacro:property name="body_center_z" value="0.428247245"/>
     <!-- Προσωρινές δυναμικές παράμετροι -->
   <xacro:property name="body_mass" value="25.0"/>
@@ -34,13 +31,13 @@
   <xacro:property name="rear_wheel_mass"   value="0.80"/>
   <xacro:property name="rear_wheel_separation" value="0.61"/>
-  <xacro:property name="rear_wheel_x" value="-0.39"/>
-  <xacro:property name="rear_wheel_z" value="-0.005"/>
+  <xacro:property name="rear_wheel_x" value="0.0"/>
+  <xacro:property name="rear_wheel_z" value="0.0"/>
   <!-- Εμπρός caster τροχοί -->
   <xacro:property name="front_wheel_radius" value="0.060"/>
   <xacro:property name="front_wheel_width"  value="0.030"/>
   <xacro:property name="front_wheel_mass"   value="0.30"/>
-  <xacro:property name="front_caster_x" value="0.24"/>
+  <xacro:property name="front_caster_x" value="0.63"/>
   <xacro:property name="front_caster_separation" value="0.38"/>
-  <xacro:property name="front_wheel_z" value="-0.040"/>
+  <xacro:property name="front_wheel_z" value="-0.035"/>
   <xacro:property name="caster_trail" value="0.03"/>
   <!-- ==================================================== -->
@@ -158,5 +155,5 @@
     <child link="base_link"/>
     <origin
-      xyz="0 0 ${base_link_height}"
+      xyz="-0.39 0 ${base_link_height}"
       rpy="0 0 0"/>
   </joint>

Commit message: Fix iWalk simulation geometry and RViz tools; enable NVIDIA graphics

File: src/iwalk_description/urdf/iwalk.urdf.xacro (robot description, xacro)
@@ -123,20 +123,12 @@
       <material name="iwalk_gray"/>
     </visual>
-    <!--
-      Για collision χρησιμοποιούμε απλή γεωμετρία.
-      Αργότερα μπορεί να αντικατασταθεί από περισσότερα boxes
-      ή από simplified collision mesh.
-    -->
+    <!-- Use the physical mesh, preserving openings instead of a solid bounding box.
+         Validate Gazebo contact performance; later replace with a simplified mesh if needed. -->
     <collision name="iwalk_body_collision">
-      <origin
-        xyz="${body_center_x}
-             ${body_center_y}
-             ${body_center_z}"
-        rpy="0 0 0"/>
+      <origin xyz="${mesh_x} ${mesh_y} ${mesh_z}"
+              rpy="${mesh_roll} ${mesh_pitch} ${mesh_yaw}"/>
       <geometry>
-        <box
-          size="${body_length}
-                ${body_width}
-                ${body_height}"/>
+        <mesh filename="package://iwalk_description/meshes/iwalk_body.STL"
+              scale="${mesh_scale} ${mesh_scale} ${mesh_scale}"/>
       </geometry>
     </collision>
@@ -150,12 +142,19 @@
       origin_z="${body_center_z}"/>
   </link>
-  <!-- base_footprint βρίσκεται στο έδαφος -->
+  <!-- Runtime-compatible root at the rear axle projection. -->
+  <link name="sim_base"/>
+  <joint name="sim_base_joint" type="fixed">
+    <parent link="sim_base"/>
+    <child link="base_link"/>
+    <origin xyz="0 0 ${base_link_height}" rpy="0 0 0"/>
+  </joint>
+  <!-- Preserve the existing footprint frame's physical position. -->
   <joint name="base_footprint_joint" type="fixed">
-    <parent link="base_footprint"/>
-    <child link="base_link"/>
-    <origin
-      xyz="-0.39 0 ${base_link_height}"
-      rpy="0 0 0"/>
+    <parent link="base_link"/>
+    <child link="base_footprint"/>
+    <origin xyz="0.39 0 ${-base_link_height}" rpy="0 0 0"/>
   </joint>
+  <xacro:include filename="sensors.xacro"/>
+  <xacro:iwalk_lidar/>
   <!-- ==================================================== -->
   <!-- REAR DRIVEN WHEELS                                   -->
